Commit message: rm namespace

File: src/go2_description/xacro/gazebo.xacro (robot description, xacro)
@@ -1,5 +1,5 @@
 <?xml version="1.0"?>
 <robot xmlns:xacro="http://www.ros.org/wiki/xacro" >
-    <xacro:macro  name="robot_gazebo_sensors" params="robot_name">
+    <xacro:macro  name="robot_gazebo_sensors">
         <gazebo>
             <plugin name="gz_ros2_control::GazeboSimROS2ControlPlugin" filename="libgz_ros2_control-system.so">

File: src/go2_description/xacro/gazebo_VLP_D435i.xacro (robot description, xacro)
@@ -1,5 +1,5 @@
 <?xml version="1.0"?>
 <robot xmlns:xacro="http://www.ros.org/wiki/xacro" >
-    <xacro:macro  name="robot_gazebo_sensors" params="robot_name">
+    <xacro:macro  name="robot_gazebo_sensors">
         <gazebo>
             <plugin name="gz_ros2_control::GazeboSimROS2ControlPlugin" filename="libgz_ros2_control-system.so">
@@ -8,5 +8,5 @@
             </plugin>
         </gazebo>
-        <ros2_control name="${robot_name}_GazeboSystem" type="system">
+        <ros2_control name="GazeboSystem" type="system">
             <hardware>
                 <plugin>gz_ros2_control/GazeboSimSystem</plugin>

File: src/go2_description/xacro/robot.xacro (robot description, xacro)
@@ -8,5 +8,5 @@
     <xacro:include filename="$(find go2_description)/xacro/gazebo.xacro"/>
     <!-- <xacro:include filename="$(find go2_description)/launch/stairs.urdf.xacro"/> -->
-    <xacro:robot_gazebo_sensors robot_name="$(arg robot_name)"/>
+    <xacro:robot_gazebo_sensors/>
     <!-- <xacro:stairs stairs="15" xpos="0" ypos="0" zpos="0" /> -->
     <!-- Rotor related joint and link is only for demonstrate location. -->

File: src/go2_description/xacro/robot_VLP_D435i.xacro (robot description, xacro)
@@ -8,5 +8,5 @@
     <xacro:include filename="$(find go2_description)/xacro/gazebo_VLP_D435i.xacro"/>
     <!-- <xacro:include filename="$(find go2_description)/launch/stairs.urdf.xacro"/> -->
-    <xacro:robot_gazebo_sensors robot_name="$(arg robot_name)"/>
+    <xacro:robot_gazebo_sensors/>
     <!-- <xacro:stairs stairs="15" xpos="0" ypos="0" zpos="0" /> -->
     <!-- Rotor related joint and link is only for demonstrate location. -->
